File: PCB/kalam.kicad_pcb (KiCad board)
At the start: 2 copper layers, 265.1 x 75.4 mm, 120 parts, among them J1 Conn_01x04, J2 Conn_01x04, U1 XC6206PxxxMR, U2 STM32F072CBTx

Commit message: PCB Fab v1
Parts:
- removed D25, D28, D42, D43, D45, D46: 1N4148W, Diode_SMD:D_SOD-123
- removed MX26, MX28, MX31, MX45, MX46, MX49, MX51: MX_SW_solder, PCM_marbastlib-mx:SW_MX_1u
- removed S3: ISO, PCM_marbastlib-mx:STAB_MX_P_ISO-ROT
- removed S4: 6.25, PCM_marbastlib-mx:STAB_MX_P_6.25u
- removed S5: 2, PCM_marbastlib-mx:STAB_MX_P_2u
- removed S6: 2.25, PCM_marbastlib-mx:STAB_MX_P_2.25u
- added REF**: Oring-Plateless-Kit, misc:Oring-Plateless-Kit, F.Cu at (206.3, 85.9)
- added REF**: Oring-Plateless-Kit, misc:Oring-Plateless-Kit, F.Cu at (81.3, 85.9)
- added REF**: Oring-Plateless-Kit, misc:Oring-Plateless-Kit, F.Cu at (60.4, 15.9)
- added REF**: Oring-Plateless-Kit, misc:Oring-Plateless-Kit, F.Cu at (213.7, 15.9)
- added S2: 2.25, PCM_marbastlib-mx:STAB_MX_P_2.25u, F.Cu at (34.2, 60.4)
- MX13: footprint PCM_marbastlib-mx:SW_MX_1.5u -> PCM_marbastlib-mx:SW_MX_1u
- MX27: footprint PCM_marbastlib-mx:SW_MX_1u -> PCM_marbastlib-mx:SW_MX_1.75u
- MX30: footprint PCM_marbastlib-mx:SW_MX_1.25u -> PCM_marbastlib-mx:SW_MX_1u
- MX41: footprint PCM_marbastlib-mx:SW_MX_1u -> PCM_marbastlib-mx:SW_MX_1.25u
- MX42: footprint PCM_marbastlib-mx:SW_MX_1.75u -> PCM_marbastlib-mx:SW_MX_1u
- S1: value 2.25 -> 6.25; footprint PCM_marbastlib-mx:STAB_MX_P_2.25u -> PCM_marbastlib-mx:STAB_MX_P_6.25u
- moved S1 120.7 mm to (143.8, 79.5)
- moved D26 9.34 mm to (244.4, 42.3), turned to 90 degrees
- moved MX30 9.23 mm to (34.2, 60.4)
- moved D13 7.56 mm to (251.8, 23.2), turned to 90 degrees
- moved MX13 5.07 mm to (260.4, 22.3)
- moved MX27 5.07 mm to (253.3, 41.4)
- moved D27 2.85 mm to (31.0, 64.0)
- moved D39 2.70 mm to (251.7, 61.2)
- moved MX42 2.70 mm to (260.4, 60.4)
- moved D38 2.10 mm to (247.0, 61.2)
- moved MX41 2.10 mm to (239.0, 60.4)
- moved D11 0.42 mm to (213.6, 23.1)
- moved D12 0.42 mm to (232.7, 23.1)
- moved D18 0.42 mm to (104.1, 42.1)
- moved D19 0.42 mm to (123.1, 42.1)
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- renumbered BOOT to SW1, RESET to SW2
Routing:
- net col5: track 197.9 -> 178.9 mm
- net Net-(D42-A): track 12.3 -> 0.00 mm
- net Net-(D27-A): track 16.2 -> 4.60 mm
- net Net-(D26-A): track 16.3 -> 4.75 mm
- net col9: track 204.5 -> 193.5 mm
- net col7: track 167.1 -> 156.3 mm
- net col0: track 89.3 -> 80.4 mm
- net Net-(D28-A): track 8.52 -> 0.00 mm
- net row1: track 298.5 -> 292.3 mm
- net col11: track 247.3 -> 241.1 mm
- net Net-(D25-A): track 5.48 -> 0.00 mm
- net Net-(D45-A): track 5.48 -> 0.00 mm
- net Net-(D46-A): track 5.48 -> 0.00 mm
- net row0: track 279.5 -> 274.0 mm
- net Net-(D43-A): track 5.45 -> 0.00 mm
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Other:
- board size 265.1 x 75.4 mm -> 256 x 75 mm
- board text added: "Caps Lock"
- board text added: "Enter"
- board text added: "Fn"
- board text added: "L.Alt"
- board text added: "L.Shift"
- board text added: "L.Super"
- board text added: "R.Alt"
- board text added: "R.Shift"
- board text added: "R.Super"
- board text added: "Space"
- board text added: "Tab"
- board text removed: "2.25u"
- board text removed: "2u"
- board text removed: "6.25u"
- board text removed: "ANSI"
- board text removed: "ISO"
- board text removed: "JLCJLCJLCJLC"
- board text removed: "STEP"

Commit message: updates
Parts:
- removed the D12 at (232.7, 23.1)
- removed the D24 at (218.4, 42.1)
- removed the D37 at (225.5, 61.2)
- removed MX12, MX25, MX40: MX_SW_solder, PCM_marbastlib-mx:SW_MX_1u
- removed REF** (x4): Oring-Plateless-Kit, misc:Oring-Plateless-Kit
- removed SW2: SW_Push, Button_Switch_SMD:SW_Push_1P1T_XKB_TS-1187A
- added S3: 2.25, PCM_marbastlib-mx:STAB_MX_P_2.25u, F.Cu at (239.0, 41.4)
- C5: value 4.7u -> 1u
- C7: value 1u -> 4.7u
- MX13: footprint PCM_marbastlib-mx:SW_MX_1u -> PCM_marbastlib-mx:SW_MX_1.5u
- MX27: footprint PCM_marbastlib-mx:SW_MX_1.75u -> PCM_marbastlib-mx:SW_MX_1u
- MX41: footprint PCM_marbastlib-mx:SW_MX_1.25u -> PCM_marbastlib-mx:SW_MX_1.75u
- MX44, MX52: footprint PCM_marbastlib-mx:SW_MX_1.5u -> PCM_marbastlib-mx:SW_MX_1.25u
- moved MX41 14.3 mm to (224.7, 60.4)
- moved D23 14.3 mm to (230.1, 42.3)
- moved MX27 14.3 mm to (239.0, 41.4)
- moved D12 14.3 mm to (237.5, 23.2)
- moved MX13 14.3 mm to (246.2, 22.3)
- moved D33 14.2 mm to (232.8, 61.2)
- moved D39 9.53 mm to (223.1, 80.2)
- moved MX53 9.53 mm to (231.9, 79.5)
- moved D34 9.52 mm to (242.2, 61.2)
- moved MX42 9.52 mm to (250.9, 60.4)
- moved D38 7.14 mm to (218.4, 80.2)
- moved MX52 7.14 mm to (210.4, 79.5)
- moved D37 4.76 mm to (130.3, 80.3)
- moved MX48 4.76 mm to (139.0, 79.5)
- moved S1 4.76 mm to (139.0, 79.5)
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- renumbered D13 to D12, D14 to D13, D15 to D14, D16 to D15, D17 to D16, D18 to D17, D19 to D18, D20 to D19, D21 to D20, D22 to D21, D23 to D22, D26 to D23, D27 to D24, D29 to D25, D30 to D26, D31 to D27, D32 to D28, D33 to D29, D34 to D30, D35 to D31, D36 to D32, D38 to D33, D39 to D34, D40 to D35, D41 to D36, D44 to D37, D47 to D38, D48 to D39
Connections:
- net RST renamed Net-(U2-NRST)
- D33 pad 2: Net-(D38-A) (its old number) -> Net-(D33-A)
- D36 pad 2: Net-(D41-A) -> Net-(D36-A)
- MX13 pad 2: col12 -> col11
- MX27 pad 2: col12 -> col11
- MX41 pad 1: Net-(D38-A) (its old number) -> col10
- MX41 pad 2: col11 -> Net-(D33-A)
- MX42 pad 2: col12 -> col11
- MX44 pad 1: Net-(D41-A) -> col2
- MX44 pad 2: col2 -> Net-(D36-A)
- U2 pad 2: col4 -> unconnected-(U2-PC13-Pad2)
- U2 pad 39: col3 -> col6
- U2 pad 40: col6 -> col7
- U2 pad 41: col7 -> col8
- U2 pad 42: col8 -> col9
- U2 pad 43: col9 -> col11
- U2 pad 45: col11 -> col4
- U2 pad 46: col12 -> col3
Routing:
- net col12: track 260.9 -> 0.00 mm
- net col11: track 241.1 -> 264.0 mm
- net Net-(U2-NRST): track 19.9 -> 2.19 mm
- net row1: track 292.3 -> 276.9 mm
- net row0: track 274.0 -> 259.8 mm
- net Net-(D38-A) (its old number): track 12.3 -> 0.00 mm
- net Net-(D37-A) (its old number): track 12.3 -> 0.00 mm
- net Net-(D41-A): track 12.3 -> 0.00 mm
- net row2_r: track 198.6 -> 188.0 mm
- net row3: track 188.2 -> 179.1 mm
- net Net-(D36-A): track 0.00 -> 9.03 mm
- net col2: track 82.4 -> 73.6 mm
- net col4: track 110.7 -> 102.1 mm
- net Net-(D33-A): track 0.00 -> 8.30 mm
- net BOOT: track 58.5 -> 51.5 mm
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Other:
- board size 256 x 75 mm -> 246.5 x 75 mm
- board text added: "BOOT"
- board text added: "designed by arko"
- board text removed: "Designed by Arko"

Commit message: back to the drawing board
Parts:
- removed J2: Conn_01x04, Connector_PinHeader_2.54mm:PinHeader_1x04_P2.54mm_Vertical
- removed the MX36 at (141.4, 60.4)
- removed the MX37 at (160.4, 60.4)
- removed the MX38 at (179.5, 60.4)
- removed the MX39 at (198.5, 60.4)
- added D40: 1N4148W, Diode_SMD:D_SOD-123, B.Cu at (156.3, 80.3)
- added D41: 1N4148W, Diode_SMD:D_SOD-123, B.Cu at (184.8, 80.2)
- added D42: 1N4148W, Diode_SMD:D_SOD-123, B.Cu at (206.3, 80.2)
- added D43: 1N4148W, Diode_SMD:D_SOD-123, B.Cu at (239.8, 80.2)
- added MX12: MX_SW_solder, PCM_marbastlib-mx:SW_MX_1.5u, F.Cu at (246.2, 22.3)
- added MX25: MX_SW_solder, PCM_marbastlib-mx:SW_MX_1u, F.Cu at (34.2, 60.4)
- added MX26: MX_SW_solder, PCM_marbastlib-mx:SW_MX_1u, F.Cu at (65.2, 60.4)
- added MX28: MX_SW_solder, PCM_marbastlib-mx:SW_MX_1u, F.Cu at (103.3, 60.4)
- added MX29: MX_SW_solder, PCM_marbastlib-mx:SW_MX_1u, F.Cu at (122.3, 60.4)
- added MX31: MX_SW_solder, PCM_marbastlib-mx:SW_MX_1u, F.Cu at (160.4, 60.4)
- added MX43: MX_SW_solder, PCM_marbastlib-mx:SW_MX_1u, F.Cu at (165.2, 79.5)
- added MX44: MX_SW_solder, PCM_marbastlib-mx:SW_MX_1.25u, F.Cu at (196.2, 79.5)
- added MX45: MX_SW_solder, PCM_marbastlib-mx:SW_MX_1u, F.Cu at (193.8, 79.5)
- added MX46: MX_SW_solder, PCM_marbastlib-mx:SW_MX_1.25u, F.Cu at (215.2, 79.5)
- added MX47: MX_SW_solder, PCM_marbastlib-mx:SW_MX_1u, F.Cu at (217.6, 79.5)
- added MX48: MX_SW_solder, PCM_marbastlib-mx:SW_MX_1.25u, F.Cu at (248.5, 79.5)
- added S4: 2, PCM_marbastlib-mx:STAB_MX_P_2u, F.Cu at (108.0, 79.5)
- added S5: 2, PCM_marbastlib-mx:STAB_MX_P_2u, F.Cu at (165.2, 79.5)
- MX13: footprint PCM_marbastlib-mx:SW_MX_1.5u -> PCM_marbastlib-mx:SW_MX_1.75u
- MX14: footprint PCM_marbastlib-mx:SW_MX_1.75u -> PCM_marbastlib-mx:SW_MX_1.75u_STP_1.25
- MX15: footprint PCM_marbastlib-mx:SW_MX_1.75u_STP_1.25 -> PCM_marbastlib-mx:SW_MX_1u
- MX34: footprint PCM_marbastlib-mx:SW_MX_1u -> PCM_marbastlib-mx:SW_MX_1.75u
- MX36: renamed from MX43; footprint PCM_marbastlib-mx:SW_MX_1u -> PCM_marbastlib-mx:SW_MX_1.25u
- MX41: footprint PCM_marbastlib-mx:SW_MX_1.75u -> PCM_marbastlib-mx:SW_MX_1u
- S1: value 6.25 -> 7; footprint PCM_marbastlib-mx:STAB_MX_P_6.25u -> PCM_marbastlib-mx:STAB_MX_P_7u
- moved MX13 217.5 mm to (29.5, 41.4)
- moved C7 158.0 mm to (218.6, 54.1), turned to 45 degrees
- moved C6 157.8 mm to (217.6, 53.2), turned to 45 degrees
- moved C2 157.6 mm to (212.3, 59.9), turned to -45 degrees
- moved MX27 155.9 mm to (84.2, 60.4)
- moved U2 155.5 mm to (211.6, 53.9), turned to 45 degrees
- moved C5 155.4 mm to (205.0, 56.9), turned to -135 degrees
- moved C4 155.2 mm to (206.2, 57.6), turned to -135 degrees
- moved SW1 154.8 mm to (239.0, 50.2)
- moved C3 152.5 mm to (211.8, 47.0), turned to 135 degrees
- moved MX40 152.4 mm to (79.5, 79.5)
- moved C10 150.9 mm to (207.4, 58.6), turned to 45 degrees
- moved C1 149.9 mm to (210.9, 47.9), turned to 135 degrees
- moved J1 148.4 mm to (198.5, 31.1), turned to 90 degrees
- moved R1 145.0 mm to (234.0, 51.3)
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- renumbered MX44 to MX37, MX48 to MX38, MX52 to MX39, MX53 to MX40
Connections:
- D24 pad 1: row2_l -> row2
- D25 pad 1: row2_r -> row2
- D26 pad 1: row2_r -> row2
- D27 pad 1: row2_r -> row2
- D28 pad 1: row2_r -> row2
- D29 pad 1: row2_r -> row2
- D30 pad 1: row2_r -> row2
- D31 pad 1: row2_r -> row2
- D32 pad 1: row2_r -> row2
- D33 pad 1: row2_r -> row2
- D34 pad 1: row2_r -> row2
- MX13 pad 1: Net-(D12-A) -> Net-(D13-A)
- MX13 pad 2: col11 -> col0
- MX14 pad 1: Net-(D13-A) -> col0
- MX14 pad 2: col0 -> Net-(D13-A)
- MX15 pad 1: col0 -> Net-(D14-A)
- MX15 pad 2: Net-(D13-A) -> col1
- MX16 pad 1: Net-(D14-A) -> Net-(D15-A)
- MX16 pad 2: col1 -> col2
- MX17 pad 1: Net-(D15-A) -> Net-(D16-A)
- MX17 pad 2: col2 -> col3
- MX18 pad 1: Net-(D16-A) -> Net-(D17-A)
- MX18 pad 2: col3 -> col4
- MX19 pad 1: Net-(D17-A) -> Net-(D18-A)
- MX19 pad 2: col4 -> col5
- MX20 pad 1: Net-(D18-A) -> Net-(D19-A)
- MX20 pad 2: col5 -> col6
- MX21 pad 1: Net-(D19-A) -> Net-(D20-A)
- MX21 pad 2: col6 -> col7
- MX22 pad 1: Net-(D20-A) -> Net-(D21-A)
- MX22 pad 2: col7 -> col8
- MX23 pad 1: Net-(D21-A) -> Net-(D22-A)
- MX23 pad 2: col8 -> col9
- MX24 pad 1: Net-(D22-A) -> Net-(D23-A)
- MX24 pad 2: col9 -> col11
- MX27 pad 1: Net-(D23-A) -> Net-(D26-A)
- MX27 pad 2: col11 -> col3
- MX30 pad 1: Net-(D24-A) -> Net-(D29-A)
- MX30 pad 2: col0 -> col6
- MX32 pad 1: Net-(D25-A) -> Net-(D31-A)
- MX32 pad 2: col2 -> col8
- MX33 pad 1: Net-(D26-A) -> Net-(D32-A)
- MX33 pad 2: col3 -> col9
- MX34 pad 1: Net-(D27-A) -> col10
- MX34 pad 2: col4 -> Net-(D33-A)
- MX35 pad 1: Net-(D28-A) -> Net-(D34-A)
- MX35 pad 2: col5 -> col11
- MX36 pad 2: col1 -> col0
- MX37 pad 1: col2 -> Net-(D36-A)
- MX37 pad 2: Net-(D36-A) -> col2
- MX38 pad 1: Net-(D37-A) -> Net-(D36-A)
- MX38 pad 2: col6 -> col2
- MX39 pad 1: Net-(D38-A) -> Net-(D37-A)
- MX39 pad 2: col10 -> col3
- MX40 pad 1: Net-(D39-A) -> Net-(D37-A)
- MX40 pad 2: col11 -> col3
- MX41 pad 1: col10 -> Net-(D38-A)
- MX41 pad 2: Net-(D33-A) -> col4
- MX42 pad 1: Net-(D34-A) -> Net-(D39-A)
- MX42 pad 2: col11 -> col6
- U2 pad 17: col1 -> unconnected-(U2-PA7-Pad17)
- U2 pad 18: row2_l -> unconnected-(U2-PB0-Pad18)
- U2 pad 19: col0 -> unconnected-(U2-PB1-Pad19)
- U2 pad 20: row1 -> unconnected-(U2-PB2-Pad20)
- U2 pad 25: row0 -> row1
- U2 pad 26: col5 -> unconnected-(U2-PB13-Pad26)
- U2 pad 27: col10 -> unconnected-(U2-PB14-Pad27)
- U2 pad 3: col2 -> row2
- U2 pad 34: SWDIO -> row0
- U2 pad 37: SWDCLK -> col10
- U2 pad 38: row2_r -> unconnected-(U2-PA15-Pad38)
- U2 pad 39: col6 -> unconnected-(U2-PB3-Pad39)
- U2 pad 4: row3 -> col9
- U2 pad 40: col7 -> unconnected-(U2-PB4-Pad40)
- U2 pad 41: col8 -> unconnected-(U2-PB5-Pad41)
- U2 pad 42: col9 -> unconnected-(U2-PB6-Pad42)
- U2 pad 43: col11 -> unconnected-(U2-PB7-Pad43)
- U2 pad 45: col4 -> unconnected-(U2-PB8-Pad45)
- U2 pad 46: col3 -> unconnected-(U2-PB9-Pad46)
Routing:
- net col10: track 295.8 -> 66.4 mm, vias 1 -> 0
- net row2: track 0.00 -> 211.9 mm, vias 0 -> 2
- net col11: track 264.0 -> 70.6 mm, vias 1 -> 0
- net row2_r: track 188.0 -> 0.00 mm
- net col5: track 180.2 -> 43.5 mm, vias 1 -> 0
- net col8: track 173.7 -> 43.5 mm, vias 1 -> 0
- net col9: track 192.9 -> 75.9 mm
- net col7: track 155.7 -> 65.9 mm, vias 1 -> 0
- net col6: track 147.2 -> 66.0 mm, vias 1 -> 0
- net row1: track 276.9 -> 203.1 mm, vias 6 -> 2
- net +3V3: track 176.9 -> 124.0 mm, vias 5 -> 8
- net SWDCLK: track 49.8 -> 0.00 mm, vias 2 -> 0
- net col1: track 67.8 -> 20.8 mm
- net SWDIO: track 46.8 -> 0.00 mm, vias 2 -> 0
- net col4: track 102.1 -> 65.8 mm, vias 1 -> 0
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Other:
- board size 246.5 x 75 mm -> 246.5 x 75.1 mm
- board text added: "2u"
- board text added: "Backspace"
- board text added: "GND D- D+ +5V"
- board text added: "L.Ctrl"
- board text added: "R.Ctrl"
- board text removed: "+5V D- D+ GND"
- board text removed: "3V3"
- board text removed: "GND"
- board text removed: "L.Alt"
- board text removed: "L.Super"
- board text removed: "R.Alt"
- board text removed: "R.Super"
- board text removed: "SWDC"
- board text removed: "SWDIO"
- board text removed: "Space"

Commit message: beeg overhaul and new layout image
Parts:
- added D35: 1N4148W, Diode_SMD:D_SOD-123, B.Cu at (242.3, 61.2)
- added MX49: MX_SW_solder, PCM_marbastlib-mx:SW_MX_1.25u, F.Cu at (215.2, 79.5)
- added MX50: MX_SW_solder, PCM_marbastlib-mx:SW_MX_1u, F.Cu at (217.6, 79.5)
- added MX51: MX_SW_solder, PCM_marbastlib-mx:SW_MX_1.25u, F.Cu at (248.5, 79.5)
- added S6: 6.25, PCM_marbastlib-mx:STAB_MX_P_6.25u, F.Cu at (124.7, 79.5)
- MX26, MX38, MX41, MX47: footprint PCM_marbastlib-mx:SW_MX_1u -> PCM_marbastlib-mx:SW_MX_1.25u
- MX34: footprint PCM_marbastlib-mx:SW_MX_1.75u -> PCM_marbastlib-mx:SW_MX_1u
- MX36: footprint PCM_marbastlib-mx:SW_MX_1.25u -> PCM_marbastlib-mx:SW_MX_1.75u
- MX37, MX44, MX46, MX48: footprint PCM_marbastlib-mx:SW_MX_1.25u -> PCM_marbastlib-mx:SW_MX_1u
- moved MX36 200.9 mm to (224.7, 60.4)
- moved MX37 193.8 mm to (250.9, 60.4)
- moved MX44 71.4 mm to (124.7, 79.5)
- moved MX43 57.1 mm to (108.0, 79.5)
- moved MX45 57.1 mm to (136.6, 79.5)
- moved MX42 57.1 mm to (79.5, 79.5)
- moved MX48 54.8 mm to (193.8, 79.5)
- moved MX35 52.4 mm to (198.5, 60.4)
- moved MX46 50.0 mm to (165.2, 79.5)
- moved MX34 45.2 mm to (179.5, 60.4)
- moved D33 43.2 mm to (189.6, 61.2)
- moved MX26 40.5 mm to (24.7, 60.4)
- moved MX31 38.1 mm to (122.3, 60.4)
- moved MX32 38.1 mm to (141.4, 60.4)
- moved MX27 38.1 mm to (46.1, 60.4)
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- renumbered D35 to D36, D36 to D37, D37 to D38, D38 to D39, D39 to D40, D40 to D41, D41 to D42, D42 to D43, D43 to D44
Connections:
- D36 pad 2: Net-(D35-A) -> Net-(D36-A)
- D37 pad 2: Net-(D36-A) -> Net-(D37-A)
- D38 pad 2: Net-(D37-A) -> Net-(D38-A)
- D39 pad 2: Net-(D38-A) -> Net-(D39-A)
- D40 pad 2: Net-(D39-A) -> Net-(D40-A)
- D41 pad 2: Net-(D40-A) -> Net-(D41-A)
- D42 pad 2: Net-(D41-A) -> Net-(D42-A)
- D43 pad 2: Net-(D42-A) -> Net-(D43-A)
- D44 pad 2: Net-(D43-A) -> Net-(D44-A)
- MX25 pad 1: col0 -> Net-(D24-A)
- MX25 pad 2: Net-(D24-A) -> col0
- MX26 pad 1: Net-(D25-A) -> Net-(D24-A)
- MX26 pad 2: col2 -> col0
- MX27 pad 1: Net-(D26-A) -> Net-(D25-A)
- MX27 pad 2: col3 -> col1
- MX28 pad 1: Net-(D27-A) -> Net-(D26-A)
- MX28 pad 2: col4 -> col2
- MX29 pad 1: Net-(D28-A) -> Net-(D27-A)
- MX29 pad 2: col5 -> col3
- MX30 pad 1: Net-(D29-A) -> Net-(D28-A)
- MX30 pad 2: col6 -> col4
- MX31 pad 1: Net-(D30-A) -> Net-(D29-A)
- MX31 pad 2: col7 -> col5
- MX32 pad 1: Net-(D31-A) -> Net-(D30-A)
- MX32 pad 2: col8 -> col6
- MX33 pad 1: Net-(D32-A) -> Net-(D31-A)
- MX33 pad 2: col9 -> col7
- MX34 pad 1: col10 -> Net-(D32-A)
- MX34 pad 2: Net-(D33-A) -> col8
- MX35 pad 1: Net-(D34-A) -> Net-(D33-A)
- MX35 pad 2: col11 -> col9
- MX36 pad 1: Net-(D35-A) -> col10
- MX36 pad 2: col0 -> Net-(D34-A)
- MX37 pad 1: Net-(D36-A) -> Net-(D35-A)
- MX37 pad 2: col2 -> col11
- MX38 pad 2: col2 -> col0
- MX39 pad 2: col3 -> col2
- MX40 pad 2: col3 -> col2
- MX41 pad 2: col4 -> col3
- MX42 pad 1: Net-(D39-A) -> Net-(D38-A)
- MX42 pad 2: col6 -> col3
- MX43 pad 1: Net-(D40-A) -> Net-(D39-A)
- MX43 pad 2: col7 -> col4
- MX44 pad 1: Net-(D41-A) -> Net-(D40-A)
- MX44 pad 2: col9 -> col6
- MX45 pad 1: Net-(D41-A) -> Net-(D40-A)
- MX45 pad 2: col9 -> col6
- MX46 pad 1: Net-(D42-A) -> Net-(D41-A)
- MX46 pad 2: col10 -> col7
- MX47 pad 2: col10 -> col9
- MX48 pad 1: Net-(D43-A) -> Net-(D42-A)
- MX48 pad 2: col11 -> col9
- U2 pad 13: unconnected-(U2-PA3-Pad13) -> col8
- U2 pad 15: unconnected-(U2-PA5-Pad15) -> col5
- U2 pad 17: unconnected-(U2-PA7-Pad17) -> col2
- U2 pad 19: unconnected-(U2-PB1-Pad19) -> col1
- U2 pad 21: unconnected-(U2-PB10-Pad21) -> col0
- U2 pad 38: unconnected-(U2-PA15-Pad38) -> col11
- U2 pad 39: unconnected-(U2-PB3-Pad39) -> row3
- U2 pad 40: unconnected-(U2-PB4-Pad40) -> col7
- U2 pad 41: unconnected-(U2-PB5-Pad41) -> col6
- U2 pad 42: unconnected-(U2-PB6-Pad42) -> col4
- U2 pad 43: unconnected-(U2-PB7-Pad43) -> col3
Routing:
- net col0: track 72.3 -> 256.9 mm, vias 0 -> 1
- net col1: track 20.8 -> 198.2 mm, vias 0 -> 1
- net col3: track 68.3 -> 205.9 mm, vias 0 -> 1
- net col2: track 70.7 -> 206.3 mm, vias 0 -> 1
- net col4: track 65.8 -> 185.7 mm, vias 0 -> 1
- net col6: track 66.0 -> 161.0 mm, vias 0 -> 1
- net col5: track 43.5 -> 122.3 mm, vias 0 -> 1
- net col7: track 65.9 -> 131.4 mm, vias 0 -> 1
- net col11: track 70.6 -> 115.5 mm, vias 0 -> 1
- net row3: track 211.6 -> 249.7 mm
- net row2: track 211.9 -> 238.9 mm
- net col8: track 43.5 -> 64.8 mm, vias 0 -> 1
- net Net-(D40-A): track 5.67 -> 24.3 mm
- net unconnected-(U2-PA15-Pad38): track 11.9 -> 0.00 mm
- net unconnected-(U2-PB3-Pad39): track 11.1 -> 0.00 mm
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Other:
- board text added: "1.25u"
- board text added: "1u"
- board text added: "6.25u"
- board text added: "7u"
- board text added: "L.Shift 2.25u"
- board text removed: "L.Shift"
